File: patchloop.kicad_pcb (KiCad board)
At the start: 2 copper layers, 36 x 39 mm, 12 parts, among them J1 8P8C, J2 Conn_Coaxial, J3 8P8C

Commit message: Minor beautification update
Parts:
- added REF**: OSHW-Logo_7.5x8mm_Copper, Symbol:OSHW-Logo_7.5x8mm_Copper, F.Cu at (129.6, 87.8)
Other:
- board text added: "CC-BY-SA 3.0"
